File: hardware/tram_tangnano/tram_tangnano.kicad_pcb (KiCad board)
At the start: 4 copper layers, 93 x 26.7 mm, 61 parts, among them J1 Conn_01x01_SolderingPad, J10 Conn_01x01_SolderingPad, J11 Conn_01x01_SolderingPad, J12 Conn_01x01_SolderingPad, J13 Conn_01x01_SolderingPad, J14 Conn_01x01_SolderingPad, J15 Conn_01x01_SolderingPad, J16 Conn_01x01_SolderingPad, J17 Conn_01x01_SolderingPad, J18 Conn_01x01_SolderingPad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

Commit message: Change to 10.x
Other:
- board text added: "V0.2 dg1vs-labs"
- board text removed: "V0.1 dg1vs-labs"
