File: hardware/tram_tangnano/tram_tangnano.kicad_pcb (KiCad board)
At the start: 4 copper layers, 93 x 26.7 mm, 40 parts, among them J1 Conn_LED, J2 Conn_Event, J3 Conn_Link, J4 Conn_Audio, U1 Tang_Nano_20K, U10 TXU0202, U11 TXU0202, U12 TXU0202, U13 TXU0202, U20 TRAM, U4 SN74LVC2GU04, U6 SN74LVC1G06, U7 SN74LVC1G04

Commit message: cleanup pluto
Parts:
- added C54: 10µF, Capacitor_SMD:C_Elec_3x5.4, F.Cu at (197.4, 102.8)
- D5: value D_Schottky_Small -> PMEG2010ER; footprint Diode_SMD:D_SMB -> Diode_SMD:Nexperia_CFP3_SOD-123W
- moved J3 2.55 mm to (214.6, 101.0)
- moved J2 2.54 mm to (214.6, 85.7)
Connections:
- J2 pad 2: /EventAck -> /EventReq
- J2 pad 3: /EventWaiting -> /EventAck
- J2 pad 4: /EventReq -> /EventWaiting
Routing:
- net Net-(D03-A1): track 16.2 -> 81.4 mm, vias 0 -> 2
- net Net-(U13-A2Y): track 0.00 -> 61.7 mm, vias 0 -> 4
- net /ExtLink2In: track 0.00 -> 59.0 mm, vias 0 -> 1
- net /ExtLink2Out: track 0.00 -> 58.9 mm, vias 0 -> 1
- net Net-(D03-A2): track 14.0 -> 59.6 mm
- net Net-(U20-Analyse): track 0.00 -> 37.7 mm, vias 0 -> 1
- net Net-(U10-A2Y): track 0.00 -> 34.3 mm, vias 0 -> 2
- net Net-(U20-Reset): track 0.01 -> 33.8 mm
- net /EventReq: track 63.5 -> 58.5 mm
- net /EventWaiting: track 61.9 -> 66.0 mm
- net +5V: track 161.2 -> 157.3 mm, vias 16 -> 17
- net +3.3V: track 161.6 -> 165.4 mm
- net Net-(U20-Link3out): track 21.0 -> 17.7 mm, vias 1 -> 0
- net GND: track 36.7 -> 39.6 mm, vias 21 -> 22
- net /ExtLink5In: track 65.1 -> 62.9 mm
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Other:
- board text added: "1"
