File: hardware/tram_tangnano/tram_tangnano.kicad_sch (KiCad schematic)
At the start: 61 parts, among them J1 Conn_01x01_SolderingPad, J10 Conn_01x01_SolderingPad, J11 Conn_01x01_SolderingPad, J12 Conn_01x01_SolderingPad, J13 Conn_01x01_SolderingPad, J14 Conn_01x01_SolderingPad, J15 Conn_01x01_SolderingPad, J16 Conn_01x01_SolderingPad, J17 Conn_01x01_SolderingPad, J18 Conn_01x01_SolderingPad, J19 Conn_01x01_SolderingPad, J2 Conn_01x01_SolderingPad, J20 Conn_01x01_SolderingPad, J21 Conn_01x01_SolderingPad, J22 Conn_01x01_SolderingPad, J23 Conn_01x01_SolderingPad, J24 Conn_01x01_SolderingPad, J3 Conn_01x04_Voltage, J4 Conn_01x01_SolderingPad, J5 Conn_01x01_SolderingPad, J6 Conn_01x01_SolderingPad, J7 Conn_01x01_SolderingPad, J8 Conn_01x01_SolderingPad, J9 Conn_01x01_SolderingPad, U1 Tang_Nano_20K, U10 TXU0202, U11 TXU0202, U12 TXU0202, U13 TXU0202, U20 TRAM, U4 SN74LVC2GU04, U6 SN74LVC1G06, U7 SN74LVC1G04

Commit message: temp
Parts:
- removed J1, J10, J11, J12, J13, J14, J15, J16, J17, J18, J19, J2, J20, J21, J22, J23, J24, J4, J5, J6, J7, J8, J9: Conn_01x01_SolderingPad, Transputer:TestPoint_THTPad_D1.5mm_Drill0.7mm, symbol Transputer:Conn_01x01_SolderingPad
- removed J3: Conn_01x04_Voltage, Transputer:PinHeader_1x04_P2.54mm_without_2, symbol Transputer:Conn_01x04_Voltage
- added J1: Conn_LED, Connector_PinHeader_2.54mm:PinHeader_1x07_P2.54mm_Vertical, symbol Connector_Generic:Conn_01x07
- added J2: Conn_Event, Connector_PinHeader_2.54mm:PinHeader_1x04_P2.54mm_Vertical, symbol Connector_Generic:Conn_01x04
- added J3: Conn_Link, Connector_PinHeader_2.54mm:PinHeader_1x06_P2.54mm_Vertical, symbol Connector_Generic:Conn_01x06
- added J4: Conn_Audio, Connector_PinHeader_2.54mm:PinHeader_1x06_P2.54mm_Vertical, symbol Connector_Generic:Conn_01x06
- C30, C31, C32, C33, C34, C35, C36, C50, C51, C52, C53: LCSC (none) -> C14663
- C59: now not fitted; now left out of the parts list
- U1, U20: now left out of the parts list
- U10, U11, U12, U13: LCSC (none) -> C7372013
Connections:
- net +5V: now also J4.6 (Pin_6)
- net GND: now also J1.1 (Pin_1), J2.1 (Pin_1), J3.1 (Pin_1), J3.4 (Pin_4), J4.5 (Pin_5)
- net ExtLink1In: now reaches U1.10 (25_IOB6A), U11.8 (B1Y)
- net ExtLink1Out: now reaches U1.11 (26_IOB6B), U11.1 (B2)
- net ExtLink2In: now reaches U1.12 (29_IOB14A)
- net ExtLink2In: now also J3.2 (Pin_2)
- net ExtLink2Out: now reaches U1.13 (30_IOB14A)
- net ExtLink2Out: now also J3.3 (Pin_3)
- net EventReq: now reaches U1.14 (31_IOB29A)
- net EventReq: now also J2.4 (Pin_4)
- net LED2: now reaches U1.15 (17_IOL49A)
- net LED2: now also J1.4 (Pin_4)
- net LED5: now reaches U1.16 (20_IOL51B)
- net LED5: now also J1.7 (Pin_7)
- net LED4: now reaches U1.17 (19_IOL51A)
- net LED4: now also J1.6 (Pin_6)
- net LED3: now reaches U1.18 (18_IOL49B)
- net LED3: now also J1.5 (Pin_5)
- net ExtLink5Out: now reaches U1.23 (71_IOT44A)
- net ExtLink5Out: now also J3.6 (Pin_6)
- net ExtLink5In: now reaches U1.24 (72_IOT40B)
- net ExtLink5In: now also J3.5 (Pin_5)
- net EventAck: now reaches U1.28 (86_IOT4A)
- net EventAck: now also J2.2 (Pin_2)
- net ExtLink4Out: now reaches U1.29 (49_IOR49A), U13.1 (B2)
- net AUDIO_I2S_LRCK: now reaches U1.30 (55_IOR36B)
- net AUDIO_I2S_LRCK: now also J4.4 (Pin_4)
- net ExtLink4In: now reaches U1.31 (48_IOR49B), U13.8 (B1Y)
- net AUDIO_PA_EN: now reaches U1.32 (51_IOR45A)
- net AUDIO_I2S_DIN: now reaches U1.33 (54_IOR38A)
- net AUDIO_I2S_DIN: now also J4.3 (Pin_3)
- net AUDIO_I2S_BCLK: now reaches U1.34 (56_IOR36A)
- net AUDIO_I2S_BCLK: now also J4.2 (Pin_2)
- net ExtLink3In: now reaches U1.35 (41_IOB43A), U12.8 (B1Y)
- net ExtLink3Out: now reaches U1.36 (42_IOB42B), U12.1 (B2)
- net EventWaiting: now reaches U1.38 (76_IOT30B)
- net EventWaiting: now also J2.3 (Pin_3)
- net LED0: now reaches U1.6 (15_IOL46A)
- net LED0: now also J1.2 (Pin_2)
- net LED1: now reaches U1.7 (16_IOL47B)
- net LED1: now also J1.3 (Pin_3)
- net ExtLink0In: now reaches U1.8 (27_IOB8A), U10.8 (B1Y)
- net ExtLink0Out: now reaches U1.9 (28_IOB8B), U10.1 (B2)
- net at R23.1, U13.5 (A1), U20.16 (Link3in): now also D03.1 (A1); no longer D03.2 (A2)
- net at R20.1, U10.5 (A1), U20.13 (Link0in): now also D03.2 (A2); no longer D03.1 (A1)
- no-connect marks 3 -> 10
Other:
- note added: "6 5 4 3 2 1"
- note removed: "Messpunkt"
- note removed: "Old! TRAM TangNano T805 T425 ------------------------------------------- Link0 Link0 Link0 Link1 Link1 Link2 Link2 Link3 Link0 Link3 Link4 Link1 Link2 Link3 Lötpunkte Link5 Link2 Lötpunkte"
- note removed: "Scottky? Wenn USB und 5V vom Board kommmen"
- company: (none) -> dg1vs-labs
- title: (none) -> TRAM-TangNano
- moved on the sheet: C30, C31, C32, C33, C34, C35, C36, C50, C51, C52, C53, D5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
