File: hardware/tram_tangnano/tram_tangnano.kicad_sch (KiCad schematic)
At the start: 41 parts, among them J1 Conn_LED, J2 Conn_Event, J3 Conn_Link, J4 Conn_Audio, U1 Tang_Nano_20K, U10 TXU0202, U11 TXU0202, U12 TXU0202, U13 TXU0202, U20 TRAM, U4 SN74LVC2GU04, U6 SN74LVC1G06, U7 SN74LVC1G04

Commit message: cleanup pluto
Parts:
- removed C59: 100µF, Capacitor_SMD:CP_Elec_5x3.9, symbol Device:C_Polarized
- added C54: 10µF, Capacitor_SMD:C_Elec_3x5.4, symbol Device:C
- D03, D21: LCSC (none) -> C68978
- D5: value D_Schottky_Small -> PMEG2010ER; footprint Diode_SMD:D_SMB -> Diode_SMD:Nexperia_CFP3_SOD-123W
- R1, R10, R11, R12, R13, R20, R21, R22, R23: LCSC (none) -> C25804
- R30, R31, R32, R33: LCSC (none) -> C25196
- U4: LCSC (none) -> C41430939
- U6: LCSC (none) -> C22469967
- U7: LCSC (none) -> C19829658
Connections:
- net +5V: now also C54.1
- net EventAck: now also J2.3 (Pin_3); no longer J2.2 (Pin_2)
- net EventReq: now also J2.2 (Pin_2); no longer J2.4 (Pin_4)
- net EventWaiting: now also J2.4 (Pin_4); no longer J2.3 (Pin_3)
- net GND: now also C54.2
Other:
- note added: "Capacitor_SMD:C_1808_4520Metric"
